File: hardware/esp32-ir-remote.kicad_pcb (KiCad board)
At the start: 2 copper layers, 0 parts

Commit message: Add circuit.md format and document ESP32 IR Remote schematic
Introduces a new markdown-based circuit description format that captures
both topology and design rationale. The format supports:
- Net and component declarations with bracket syntax
- Inline passives: [VCC --- 10kΩ --- EN]
- Design properties: [dropout ==> 1.2V]
- Subcircuit references: @./power-supply.circuit.md

Circuit documentation for ESP32 IR Remote board:
- power-supply.circuit.md: USB-C, protection, AP63203 buck
- usb-serial.circuit.md: CH340C with auto-reset circuit
- esp32-mcu.circuit.md: ESP32-WROOM-32E module
- ir-transmitter.circuit.md: 4x TSAL6200 with MOSFET driver
- ir-receiver.circuit.md: TSOP38238 for development
- temp-sensor.circuit.md: DHT22/AM2302
- status-leds.circuit.md: Serial and user indicators

Also includes:
- Parser and KiCad export scripts
- Component datasheets
- Updated schematic and PCB layout
- BOM export

🤖 Generated with [Claude Code](https://claude.com/claude-code)

Co-Authored-By: Claude Opus 4.5 <noreply@anthropic.com>
Parts:
- added C1: 10µF, Capacitor_SMD:C_0805_2012Metric, F.Cu at (109.7, 102.5)
- added C10: 100nF, Capacitor_SMD:C_0603_1608Metric, F.Cu at (136.2, 106.5)
- added C2: 22µF, Capacitor_SMD:C_0805_2012Metric, F.Cu at (109.7, 105.5)
- added C3: 22µF, Capacitor_SMD:C_0805_2012Metric, F.Cu at (109.7, 108.5)
- added C4: 100nF, Capacitor_SMD:C_0603_1608Metric, F.Cu at (127.3, 102.3)
- added C5: 100nF, Capacitor_SMD:C_0603_1608Metric, F.Cu at (127.3, 104.8)
- added C6: 1µF, Capacitor_SMD:C_0805_2012Metric, F.Cu at (109.7, 111.5)
- added C7: 100nF, Capacitor_SMD:C_0603_1608Metric, F.Cu at (127.3, 107.3)
- added C8: 10µF, Capacitor_SMD:C_0805_2012Metric, F.Cu at (109.7, 114.5)
- added C9: 100nF, Capacitor_SMD:C_0603_1608Metric, F.Cu at (127.3, 109.8)
- added D1: D_TVS, Diode_SMD:D_SMB, F.Cu at (89.3, 115.8)
- added D10: Red, LED_THT:LED_D3.0mm, F.Cu at (92.7, 93.9)
- added D11: Blue, LED_THT:LED_D3.0mm, F.Cu at (92.7, 99.4)
- added D12: Blue, LED_THT:LED_D3.0mm, F.Cu at (92.7, 104.8)
- added D2: TSAL6200, LED_THT:LED_D5.0mm, F.Cu at (120.3, 52.4)
- added D3: TSAL6200, LED_THT:LED_D5.0mm, F.Cu at (120.3, 59.8)
- added D4: TSAL6200, LED_THT:LED_D5.0mm, F.Cu at (120.3, 67.3)
- added D5: TSAL6200, LED_THT:LED_D5.0mm, F.Cu at (120.3, 74.8)
- added D6: Red, LED_THT:LED_D3.0mm, F.Cu at (86.8, 93.9)
- added D7: Green, LED_THT:LED_D3.0mm, F.Cu at (86.8, 99.4)
- added D8: Amber, LED_THT:LED_D3.0mm, F.Cu at (86.8, 104.8)
- added D9: Amber, LED_THT:LED_D3.0mm, F.Cu at (86.8, 110.3)
- added F1: 1.1A, Fuse:Fuse_1812_4532Metric, F.Cu at (64.6, 101.4)
- added J1: ESP32-WROOM-32E-Breakout, lib:PinHeader_2x19_P2.54mm_DevKitC, F.Cu at (63.4, 50.9)
- added J2: USB_C_Receptacle_USB2.0_14P, Connector_USB:USB_C_Receptacle_GCT_USB4085, F.Cu at (120.7, 80.1)
- added JP1: Buck Disable, TestPoint:TestPoint_2Pads_Pitch2.54mm_Drill0.8mm, F.Cu at (63.0, 105.6)
- added L1: 3.9µH, lib:INDM5752X300N, F.Cu at (121.1, 116.0)
- added Q1: Q_NPN_BCE, Package_TO_SOT_SMD:SOT-23, F.Cu at (114.3, 103.2)
- added Q2: Q_NPN_BCE, Package_TO_SOT_SMD:SOT-23, F.Cu at (114.3, 107.7)
- added Q3: IRLML6344, Package_TO_SOT_SMD:SOT-23, F.Cu at (114.3, 112.1)
- added Q4: 2N7002, PCM_JLCPCB:Q_SOT-23, F.Cu at (96.4, 127.6)
- added Q5: 2N7002, PCM_JLCPCB:Q_SOT-23, F.Cu at (96.4, 132.2)
- added R1: 5.1kΩ, Resistor_SMD:R_1206_3216Metric, F.Cu at (71.1, 92.8)
- added R10: 18Ω, Resistor_SMD:R_1206_3216Metric, F.Cu at (76.7, 96.1)
- added R11: 18Ω, Resistor_SMD:R_1206_3216Metric, F.Cu at (76.7, 99.4)
- added R12: 18Ω, Resistor_SMD:R_1206_3216Metric, F.Cu at (76.7, 102.7)
- added R13: 10kΩ, Resistor_SMD:R_1206_3216Metric, F.Cu at (76.7, 106.0)
- added R14: 100kΩ, Resistor_SMD:R_1206_3216Metric, F.Cu at (76.7, 109.4)
- added R15: 1kΩ, Resistor_SMD:R_1206_3216Metric, F.Cu at (76.7, 112.7)
- added R16: 150Ω, Resistor_SMD:R_1206_3216Metric, F.Cu at (76.7, 116.0)
- added R17: 470Ω, Resistor_SMD:R_1206_3216Metric, F.Cu at (82.3, 92.8)
- added R18: 470Ω, Resistor_SMD:R_1206_3216Metric, F.Cu at (82.3, 96.1)
- added R19: 470Ω, Resistor_SMD:R_1206_3216Metric, F.Cu at (82.3, 99.4)
- added R2: 5.1kΩ, Resistor_SMD:R_1206_3216Metric, F.Cu at (71.1, 96.1)
- added R20: 1kΩ, PCM_JLCPCB:R_0805, F.Cu at (101.1, 126.7)
- added R21: 0Ω, PCM_JLCPCB:R_0603, F.Cu at (59.7, 119.8)
- added R22: 10kΩ, Resistor_SMD:R_1206_3216Metric, F.Cu at (82.3, 109.4)
- added R23: 100kΩ, PCM_JLCPCB:R_0603, F.Cu at (100.7, 132.2)
- added R24: 100kΩ, PCM_JLCPCB:R_0603, F.Cu at (100.7, 134.5)
- added R25: 1kΩ, PCM_JLCPCB:R_0805, F.Cu at (101.1, 129.7)
- added R26: 0Ω, PCM_JLCPCB:R_0603, F.Cu at (59.7, 122.0)
- added R3: 10kΩ, Resistor_SMD:R_1206_3216Metric, F.Cu at (71.1, 99.4)
- added R4: 10kΩ, Resistor_SMD:R_1206_3216Metric, F.Cu at (71.1, 102.7)
- added R5: 10kΩ, Resistor_SMD:R_1206_3216Metric, F.Cu at (71.1, 106.0)
- added R6: 10kΩ, Resistor_SMD:R_1206_3216Metric, F.Cu at (71.1, 109.4)
- added R7: 10kΩ, Resistor_SMD:R_1206_3216Metric, F.Cu at (71.1, 112.7)
- added R8: 10kΩ, Resistor_SMD:R_1206_3216Metric, F.Cu at (71.1, 116.0)
- added R9: 18Ω, Resistor_SMD:R_1206_3216Metric, F.Cu at (76.7, 92.8)
- added SW1: RESET, Button_Switch_THT:SW_PUSH_6mm, F.Cu at (98.9, 103.0)
- added SW2: BOOT, Button_Switch_THT:SW_PUSH_6mm, F.Cu at (98.9, 111.6)
- added U1: AP63203WU, Package_TO_SOT_SMD:TSOT-23-6, F.Cu at (63.7, 109.6)
- added U2: CH340C, Package_SO:SOIC-16_3.9x9.9mm_P1.27mm, F.Cu at (121.0, 106.9)
- added U3: ESP32-WROOM-32E, RF_Module:ESP32-WROOM-32D, F.Cu at (93.1, 80.1)
- added U4: TSOP382xx, OptoDevice:Vishay_MINICAST-3Pin, F.Cu at (125.2, 93.3)
- added U5: AM2302, Sensor:ASAIR_AM2302_P2.54mm_Vertical, F.Cu at (101.8, 94.7)
